Commit message: Big reorganization and cleanup.

File: hexapod_description/model/gen_tetrapod.urdf.xacro (robot description, xacro)
@@ -3,3 +3,4 @@
   <xacro:include filename="$(arg model_path)/tetrapod.urdf.xacro"/>
   <xacro:tetrapod/>
+  <xacro:include filename="$(find hexapod_description)/model/common.gazebo.xacro"/>
 </robot>

File: hexapod_description/model/leg.gazebo.xacro (robot description, xacro)
@@ -2,25 +2,4 @@
 <robot xmlns:xacro="http://ros.org/wiki/xacro">
   <xacro:macro name="hexapod_leg_gazebo" params="name">
-    <gazebo>
-      <plugin name="gazebo_ros_control" filename="libgazebo_ros_control.so">
-        <robotNamespace>/${name}_leg</robotNamespace>
-      </plugin>
-    </gazebo>
-    <gazebo reference="${name}_leg_base_link">
-      <gravity>true</gravity>
-      <selfCollide>true</selfCollide>
-    </gazebo>
-    <gazebo reference="${name}_leg_link_0">
-      <gravity>true</gravity>
-      <selfCollide>true</selfCollide>
-    </gazebo>
-    <gazebo reference="${name}_leg_link_1">
-      <gravity>true</gravity>
-      <selfCollide>true</selfCollide>
-    </gazebo>
-    <gazebo reference="${name}_leg_link_2">
-      <gravity>true</gravity>
-      <selfCollide>true</selfCollide>
-    </gazebo>
   </xacro:macro>
 </robot>

File: hexapod_description/model/leg.urdf.xacro (robot description, xacro)
@@ -30,10 +30,11 @@
       </inertial>
     </link>
-    <!-- TODO: change ALL joints to revolute and add limits! -->
-    <joint name="${name}_leg_joint_0" type="continuous">
+    <!-- TODO: change ALL joints to add correct limits! -->
+    <joint name="${name}_leg_joint_0" type="revolute">
       <parent link="${name}_leg_base_link"/>
       <child link="${name}_leg_link_0"/>
       <origin xyz="0.036 0 0" rpy="0 0 0"/>
       <axis xyz="0 0 1"/>
+      <limit lower="-1.57" upper="1.57" velocity="1.57" effort="1000"/>
     </joint>
     <link name="${name}_leg_link_0">
@@ -71,9 +72,10 @@
       </inertial>
     </link>
-    <joint name="${name}_leg_joint_1" type="continuous">
+    <joint name="${name}_leg_joint_1" type="revolute">
       <parent link="${name}_leg_link_0"/>
       <child link="${name}_leg_link_1"/>
       <origin xyz="0.049 0 -0.0145" rpy="0 0 0"/>
       <axis xyz="0 1 0"/>
+      <limit lower="-1.57" upper="1.57" velocity="1.57" effort="1000"/>
     </joint>
     <link name="${name}_leg_link_1">
@@ -135,9 +137,10 @@
       </inertial>
     </link>
-    <joint name="${name}_leg_joint_2" type="continuous">
+    <joint name="${name}_leg_joint_2" type="revolute">
       <parent link="${name}_leg_link_1"/>
       <child link="${name}_leg_link_2"/>
       <origin xyz="0.0605 0 -0.0225" rpy="0 0 0"/>
       <axis xyz="0 -1 0"/>
+      <limit lower="-1.57" upper="1.57" velocity="1.57" effort="1000"/>
     </joint>
     <link name="${name}_leg_link_2">
