Commit message: Complete single leg URDF/xacro model.

File: hexapod_description/model/leg.urdf.xacro (robot description, xacro)
@@ -11,4 +11,5 @@
       </visual>
     </link>
+    <!-- TODO: change ALL joints to revolute and add limits! -->
     <joint name="${name}_leg_joint_0" type="continuous">
       <parent link="${name}_leg_base_link"/>
@@ -24,4 +25,62 @@
         </geometry>
       </visual>
+      <visual>
+        <origin xyz="0.049 0 -0.0145" rpy="${pi/2} 0 ${-pi/2}"/>
+        <geometry>
+          <mesh filename="package://hexapod_description/meshes/F1.dae" scale="0.001 0.001 0.001"/>
+        </geometry>
+      </visual>
+    </link>
+    <joint name="${name}_leg_joint_1" type="continuous">
+      <parent link="${name}_leg_link_0"/>
+      <child link="${name}_leg_link_1"/>
+      <origin xyz="0.049 0 -0.0145" rpy="0 0 0"/>
+      <axis xyz="0 1 0"/>
+    </joint>
+    <link name="${name}_leg_link_1">
+      <visual>
+        <origin xyz="0 0 0" rpy="${pi/2} ${-pi/2x} 0"/>
+        <geometry>
+          <mesh filename="package://hexapod_description/meshes/AX12.dae" scale="0.001 0.001 0.001"/>
+        </geometry>
+      </visual>
+      <visual>
+        <origin xyz="0.0415 0 0" rpy="0 ${-pi/2} ${pi/2x}"/>
+        <geometry>
+          <mesh filename="package://hexapod_description/meshes/F3.dae" scale="0.001 0.001 0.001"/>
+        </geometry>
+      </visual>
+      <visual>
+        <origin xyz="0.0415 0 0" rpy="0 ${-pi/2} ${-pi/2x}"/>
+        <geometry>
+          <mesh filename="package://hexapod_description/meshes/F3.dae" scale="0.001 0.001 0.001"/>
+        </geometry>
+      </visual>
+      <visual>
+        <origin xyz="0.0605 0 -0.0225" rpy="${-pi/2} 0 ${pi}"/>
+        <geometry>
+          <mesh filename="package://hexapod_description/meshes/AX12.dae" scale="0.001 0.001 0.001"/>
+        </geometry>
+      </visual>
+    </link>
+    <joint name="${name}_leg_joint_2" type="continuous">
+      <parent link="${name}_leg_link_1"/>
+      <child link="${name}_leg_link_2"/>
+      <origin xyz="0.0605 0 -0.0225" rpy="0 0 0"/>
+      <axis xyz="0 -1 0"/>
+    </joint>
+    <link name="${name}_leg_link_2">
+      <visual>
+        <origin xyz="0 0 0" rpy="${pi} 0 ${pi/2x}"/>
+        <geometry>
+          <mesh filename="package://hexapod_description/meshes/F4.dae" scale="0.001 0.001 0.001"/>
+        </geometry>
+      </visual>
+      <visual>
+        <origin xyz="0.0135 0 -0.055" rpy="${pi/2} ${-pi/2} 0"/>
+        <geometry>
+          <mesh filename="package://hexapod_description/meshes/F6.dae" scale="0.001 0.001 0.001"/>
+        </geometry>
+      </visual>
     </link>
   </xacro:macro>

Commit message: Add collision and inertial elements to links.

File: hexapod_description/model/leg.urdf.xacro (robot description, xacro)
@@ -2,4 +2,7 @@
 <robot xmlns:xacro="http://www.ros.org/wiki/xacro" name="leg">
   <xacro:property name="pi" value="3.1415926535897931"/>
+  <!-- VERY ROUGH ESTIMATES OF THE MASS OF THE SERVOS AND THE PLASTIC LINKAGES -->
+  <xacro:property name="AX12_m" value="0.05"/>
+  <xacro:property name="LINKAGE_m" value="0.02"/>
   <xacro:macro name="leg" params="name">
     <link name="${name}_leg_base_link">
@@ -10,4 +13,18 @@
         </geometry>
       </visual>
+      <collision>
+        <origin xyz="0.036 0 0" rpy="0 0 ${-pi/2}"/>
+        <geometry>
+          <mesh filename="package://hexapod_description/meshes/AX12.dae" scale="0.001 0.001 0.001"/>
+        </geometry>
+      </collision>
+      <inertial>
+        <origin xyz="-0.0135 0 0" rpy="0 0 0"/>
+        <mass value="${AX12_m}"/>
+        <inertia
+          ixx="1.0" ixy="0.0" ixz="0.0"
+          iyy="1.0" iyz="0.0"
+          izz="1.0"/>
+      </inertial>
     </link>
     <!-- TODO: change ALL joints to revolute and add limits! -->
@@ -31,4 +48,24 @@
         </geometry>
       </visual>
+      <collision>
+        <origin xyz="0 0 0" rpy="0 ${pi/2} 0"/>
+        <geometry>
+          <mesh filename="package://hexapod_description/meshes/F2.dae" scale="0.001 0.001 0.001"/>
+        </geometry>
+      </collision>
+      <collision>
+        <origin xyz="0.049 0 -0.0145" rpy="${pi/2} 0 ${-pi/2}"/>
+        <geometry>
+          <mesh filename="package://hexapod_description/meshes/F1.dae" scale="0.001 0.001 0.001"/>
+        </geometry>
+      </collision>
+      <inertial>
+        <origin xyz="0.026 0 0" rpy="0 0 0"/>
+        <mass value="${2*LINKAGE_m}"/>
+        <inertia
+          ixx="1.0" ixy="0.0" ixz="0.0"
+          iyy="1.0" iyz="0.0"
+          izz="1.0"/>
+      </inertial>
     </link>
     <joint name="${name}_leg_joint_1" type="continuous">
@@ -63,4 +100,36 @@
         </geometry>
       </visual>
+      <collision>
+        <origin xyz="0 0 0" rpy="${pi/2} ${-pi/2x} 0"/>
+        <geometry>
+          <mesh filename="package://hexapod_description/meshes/AX12.dae" scale="0.001 0.001 0.001"/>
+        </geometry>
+      </collision>
+      <collision>
+        <origin xyz="0.0415 0 0" rpy="0 ${-pi/2} ${pi/2x}"/>
+        <geometry>
+          <mesh filename="package://hexapod_description/meshes/F3.dae" scale="0.001 0.001 0.001"/>
+        </geometry>
+      </collision>
+      <collision>
+        <origin xyz="0.0415 0 0" rpy="0 ${-pi/2} ${-pi/2x}"/>
+        <geometry>
+          <mesh filename="package://hexapod_description/meshes/F3.dae" scale="0.001 0.001 0.001"/>
+        </geometry>
+      </collision>
+      <collision>
+        <origin xyz="0.0605 0 -0.0225" rpy="${-pi/2} 0 ${pi}"/>
+        <geometry>
+          <mesh filename="package://hexapod_description/meshes/AX12.dae" scale="0.001 0.001 0.001"/>
+        </geometry>
+      </collision>
+      <inertial>
+        <origin xyz="0.04275 0 -0.01125" rpy="0 0 0"/>
+        <mass value="${2*AX12_m + 2*LINKAGE_m}"/>
+        <inertia
+          ixx="1.0" ixy="0.0" ixz="0.0"
+          iyy="1.0" iyz="0.0"
+          izz="1.0"/>
+      </inertial>
     </link>
     <joint name="${name}_leg_joint_2" type="continuous">
@@ -83,4 +152,24 @@
         </geometry>
       </visual>
+      <collision>
+        <origin xyz="0 0 0" rpy="${pi} 0 ${pi/2x}"/>
+        <geometry>
+          <mesh filename="package://hexapod_description/meshes/F4.dae" scale="0.001 0.001 0.001"/>
+        </geometry>
+      </collision>
+      <collision>
+        <origin xyz="0.0135 0 -0.055" rpy="${pi/2} ${-pi/2} 0"/>
+        <geometry>
+          <mesh filename="package://hexapod_description/meshes/F6.dae" scale="0.001 0.001 0.001"/>
+        </geometry>
+      </collision>
+      <inertial>
+        <origin xyz="0 0 -0.05" rpy="0 0 0"/>
+        <mass value="${2*LINKAGE_m}"/>
+        <inertia
+          ixx="1.0" ixy="0.0" ixz="0.0"
+          iyy="1.0" iyz="0.0"
+          izz="1.0"/>
+      </inertial>
     </link>
   </xacro:macro>

Commit message: TMP improve collision and inertial elements. Start documenting.

File: hexapod_description/model/leg.urdf.xacro (robot description, xacro)
@@ -16,7 +16,7 @@
       </visual>
       <collision>
-        <origin xyz="0.036 0 0" rpy="0 0 ${-pi/2}"/>
-        <geometry>
-          <mesh filename="package://hexapod_description/meshes/AX12.dae" scale="0.001 0.001 0.001"/>
+        <origin xyz="0.0225 0 0" rpy="0 0 0"/>
+        <geometry>
+          <box size="0.05 0.026 0.032"/>
         </geometry>
       </collision>
@@ -25,7 +25,7 @@
         <mass value="${AX12_m}"/>
         <inertia
-          ixx="1.0" ixy="0.0" ixz="0.0"
-          iyy="1.0" iyz="0.0"
-          izz="1.0"/>
+          ixx="1.0e-6" ixy="0.0" ixz="0.0"
+          iyy="1.0e-6" iyz="0.0"
+          izz="1.0e-6"/>
       </inertial>
     </link>
@@ -50,14 +50,40 @@
         </geometry>
       </visual>
-      <collision>
-        <origin xyz="0 0 0" rpy="0 ${pi/2} 0"/>
-        <geometry>
-          <mesh filename="package://hexapod_description/meshes/F2.dae" scale="0.001 0.001 0.001"/>
-        </geometry>
-      </collision>
-      <collision>
-        <origin xyz="0.049 0 -0.0145" rpy="${pi/2} 0 ${-pi/2}"/>
-        <geometry>
-          <mesh filename="package://hexapod_description/meshes/F1.dae" scale="0.001 0.001 0.001"/>
+      <!-- F2 simplified -->
+      <collision>
+        <origin xyz="0.013 0 0.0225" rpy="0 0 0"/>
+        <geometry>
+          <box size="0.026 0.025 0.003"/>
+        </geometry>
+      </collision>
+      <collision>
+        <origin xyz="0.013 0 -0.0225" rpy="0 0 0"/>
+        <geometry>
+          <box size="0.026 0.025 0.003"/>
+        </geometry>
+      </collision>
+      <collision>
+        <origin xyz="0.0235 0 0" rpy="0 0 0"/>
+        <geometry>
+          <box size="0.005 0.025 0.048"/>
+        </geometry>
+      </collision>
+      <!-- F1 simplified -->
+      <collision>
+        <origin xyz="0.0375 0.0225 -0.001" rpy="0 0 0"/>
+        <geometry>
+          <box size="0.023 0.003 0.027"/>
+        </geometry>
+      </collision>
+      <collision>
+        <origin xyz="0.0375 -0.0225 -0.001" rpy="0 0 0"/>
+        <geometry>
+          <box size="0.023 0.003 0.027"/>
+        </geometry>
+      </collision>
+      <collision>
+        <origin xyz="0.0285 0 0" rpy="0 0 0"/>
+        <geometry>
+          <box size="0.005 0.048 0.025"/>
         </geometry>
       </collision>
@@ -66,7 +92,7 @@
         <mass value="${2*LINKAGE_m}"/>
         <inertia
-          ixx="1.0" ixy="0.0" ixz="0.0"
-          iyy="1.0" iyz="0.0"
-          izz="1.0"/>
+          ixx="1.0e-6" ixy="0.0" ixz="0.0"
+          iyy="1.0e-6" iyz="0.0"
+          izz="1.0e-6"/>
       </inertial>
     </link>
@@ -130,7 +156,7 @@
         <mass value="${2*AX12_m + 2*LINKAGE_m}"/>
         <inertia
-          ixx="1.0" ixy="0.0" ixz="0.0"
-          iyy="1.0" iyz="0.0"
-          izz="1.0"/>
+          ixx="1.0e-6" ixy="0.0" ixz="0.0"
+          iyy="1.0e-6" iyz="0.0"
+          izz="1.0e-6"/>
       </inertial>
     </link>
@@ -170,7 +196,7 @@
         <mass value="${2*LINKAGE_m}"/>
         <inertia
-          ixx="1.0" ixy="0.0" ixz="0.0"
-          iyy="1.0" iyz="0.0"
-          izz="1.0"/>
+          ixx="1.0e-6" ixy="0.0" ixz="0.0"
+          iyy="1.0e-6" iyz="0.0"
+          izz="1.0e-6"/>
       </inertial>
     </link>

File: hexapod_description/model/tetrapod.urdf.xacro (robot description, xacro)
@@ -36,7 +36,7 @@
       <mass value="0.04"/>
       <inertia
-        ixx="1.0" ixy="0.0" ixz="0.0"
-        iyy="1.0" iyz="0.0"
-        izz="1.0"/>
+        ixx="1.0E-6" ixy="0.0" ixz="0.0"
+        iyy="1.0E-6" iyz="0.0"
+        izz="1.0E-6"/>
     </inertial>
   </link>

Commit message: Simplify collision meshes by computing convex hull with meshlab.

File: hexapod_description/model/leg.urdf.xacro (robot description, xacro)
@@ -18,5 +18,5 @@
         <origin xyz="0.036 0 0" rpy="0 0 ${-pi/2}"/>
         <geometry>
-          <mesh filename="package://hexapod_description/meshes/AX12.dae" scale="0.001 0.001 0.001"/>
+          <mesh filename="package://hexapod_description/meshes/AX12_collision.dae" scale="0.001 0.001 0.001"/>
         </geometry>
       </collision>
@@ -54,5 +54,5 @@
         <origin xyz="0 0 0" rpy="0 ${pi/2} 0"/>
         <geometry>
-          <mesh filename="package://hexapod_description/meshes/F2.dae" scale="0.001 0.001 0.001"/>
+          <mesh filename="package://hexapod_description/meshes/F2_collision.dae" scale="0.001 0.001 0.001"/>
         </geometry>
       </collision>
@@ -60,5 +60,5 @@
         <origin xyz="0.049 0 -0.0145" rpy="${pi/2} 0 ${-pi/2}"/>
         <geometry>
-          <mesh filename="package://hexapod_description/meshes/F1.dae" scale="0.001 0.001 0.001"/>
+          <mesh filename="package://hexapod_description/meshes/F1_collision.dae" scale="0.001 0.001 0.001"/>
         </geometry>
       </collision>
@@ -107,5 +107,5 @@
         <origin xyz="0 0 0" rpy="${pi/2} ${-pi/2x} 0"/>
         <geometry>
-          <mesh filename="package://hexapod_description/meshes/AX12.dae" scale="0.001 0.001 0.001"/>
+          <mesh filename="package://hexapod_description/meshes/AX12_collision.dae" scale="0.001 0.001 0.001"/>
         </geometry>
       </collision>
@@ -113,5 +113,5 @@
         <origin xyz="0.0415 0 0" rpy="0 ${-pi/2} ${pi/2x}"/>
         <geometry>
-          <mesh filename="package://hexapod_description/meshes/F3.dae" scale="0.001 0.001 0.001"/>
+          <mesh filename="package://hexapod_description/meshes/F3_collision.dae" scale="0.001 0.001 0.001"/>
         </geometry>
       </collision>
@@ -119,5 +119,5 @@
         <origin xyz="0.0415 0 0" rpy="0 ${-pi/2} ${-pi/2x}"/>
         <geometry>
-          <mesh filename="package://hexapod_description/meshes/F3.dae" scale="0.001 0.001 0.001"/>
+          <mesh filename="package://hexapod_description/meshes/F3_collision.dae" scale="0.001 0.001 0.001"/>
         </geometry>
       </collision>
@@ -125,5 +125,5 @@
         <origin xyz="0.0605 0 -0.0225" rpy="${-pi/2} 0 ${pi}"/>
         <geometry>
-          <mesh filename="package://hexapod_description/meshes/AX12.dae" scale="0.001 0.001 0.001"/>
+          <mesh filename="package://hexapod_description/meshes/AX12_collision.dae" scale="0.001 0.001 0.001"/>
         </geometry>
       </collision>
@@ -160,5 +160,5 @@
         <origin xyz="0 0 0" rpy="${pi} 0 ${pi/2x}"/>
         <geometry>
-          <mesh filename="package://hexapod_description/meshes/F4.dae" scale="0.001 0.001 0.001"/>
+          <mesh filename="package://hexapod_description/meshes/F4_collision.dae" scale="0.001 0.001 0.001"/>
         </geometry>
       </collision>
@@ -166,5 +166,5 @@
         <origin xyz="0.0135 0 -0.055" rpy="${pi/2} ${-pi/2} 0"/>
         <geometry>
-          <mesh filename="package://hexapod_description/meshes/F6.dae" scale="0.001 0.001 0.001"/>
+          <mesh filename="package://hexapod_description/meshes/F6_collision.dae" scale="0.001 0.001 0.001"/>
         </geometry>
       </collision>
