Commit message: Fix collision meshes.

File: hexapod_description/scad/body.cog.urdf.xacro (robot description, xacro)
@@ -35,5 +35,23 @@
       <origin xyz="0 0 0" rpy="0 0 0"/>
       <geometry>
-        <mesh filename="package://hexapod_description/meshes/body.dae" scale="0.001 0.001 0.001"/>
+        <!--[[[cog
+        import cog
+        cog.outl('<mesh filename="file://{0}" scale="0.001 0.001 0.001"/>'.format(FILENAME))
+        ]]]-->
+        <!--[[[end]]]-->
+      </geometry>
+    </collision>
+    <collision>
+      <!--[[[cog
+      import cog
+      cog.outl('<origin xyz="0 0 {0}" rpy="0 0 0"/>'.format( (float(H)+32)/1000.0 ))
+      ]]]-->
+      <!--[[[end]]]-->
+      <geometry>
+        <!--[[[cog
+        import cog
+        cog.outl('<mesh filename="file://{0}" scale="0.001 0.001 0.001"/>'.format(FILENAME))
+        ]]]-->
+        <!--[[[end]]]-->
       </geometry>
     </collision>

Commit message: Add material for gray color.

File: hexapod_description/scad/body.cog.urdf.xacro (robot description, xacro)
@@ -17,4 +17,7 @@
         <!--[[[end]]]-->
       </geometry>
+      <material name="gray">
+        <color rgba="0.7 0.7 0.7 1"/>
+      </material>
     </visual>
     <visual>
@@ -31,4 +34,7 @@
         <!--[[[end]]]-->
       </geometry>
+      <material name="gray">
+        <color rgba="0.7 0.7 0.7 1"/>
+      </material>
     </visual>
     <collision>

Commit message: Rename links in generated URDF.

File: hexapod_description/scad/body.cog.urdf.xacro (robot description, xacro)
@@ -3,9 +3,9 @@
   <xacro:include filename="$(find hexapod_description)/model/leg.urdf.xacro"/>
   <link name="base_link"/>
-  <joint name="test_body_base_joint" type="fixed">
+  <joint name="body_joint" type="fixed">
     <parent link="base_link"/>
-    <child link="test_body_base_link"/>
+    <child link="body_link"/>
   </joint>
-  <link name="test_body_base_link">
+  <link name="body_link">
     <visual>
       <origin xyz="0 0 0" rpy="0 0 0"/>
@@ -71,7 +71,7 @@
     </inertial>
   </link>
-  <joint name="test_body_fr_leg_joint" type="fixed">
-    <parent link="test_body_base_link"/>
-    <child link="test_body_fr_leg_base_link"/>
+  <joint name="fr_leg_joint" type="fixed">
+    <parent link="body_link"/>
+    <child link="fr_leg_base_link"/>
     <!--[[[cog
     import cog
@@ -80,8 +80,8 @@
     <!--[[[end]]]-->
   </joint>
-  <xacro:leg name="test_body_fr"/>
-  <joint name="test_body_rr_leg_joint" type="fixed">
-    <parent link="test_body_base_link"/>
-    <child link="test_body_rr_leg_base_link"/>
+  <xacro:leg name="fr"/>
+  <joint name="rr_leg_joint" type="fixed">
+    <parent link="body_link"/>
+    <child link="rr_leg_base_link"/>
     <!--[[[cog
     import cog
@@ -90,8 +90,8 @@
     <!--[[[end]]]-->
   </joint>
-  <xacro:leg name="test_body_rr"/>
-  <joint name="test_body_rl_leg_joint" type="fixed">
-    <parent link="test_body_base_link"/>
-    <child link="test_body_rl_leg_base_link"/>
+  <xacro:leg name="rr"/>
+  <joint name="rl_leg_joint" type="fixed">
+    <parent link="body_link"/>
+    <child link="rl_leg_base_link"/>
     <!--[[[cog
     import cog
@@ -100,8 +100,8 @@
     <!--[[[end]]]-->
   </joint>
-  <xacro:leg name="test_body_rl"/>
-  <joint name="test_body_fl_leg_joint" type="fixed">
-    <parent link="test_body_base_link"/>
-    <child link="test_body_fl_leg_base_link"/>
+  <xacro:leg name="rl"/>
+  <joint name="fl_leg_joint" type="fixed">
+    <parent link="body_link"/>
+    <child link="fl_leg_base_link"/>
     <!--[[[cog
     import cog
@@ -110,4 +110,4 @@
     <!--[[[end]]]-->
   </joint>
-  <xacro:leg name="test_body_fl"/>
+  <xacro:leg name="fl"/>
 </robot>
